File: KiCad/IIeAux.kicad_sch (KiCad schematic)
At the start: 21 parts, among them J1 Apple IIe Aux, J4 PAL, U1 SN74LVC245AN, U2 TangNano9K, U3 74LS245, U4 74LS374, U5 SN74LVC245AN, U6 SN74LVC245AN, U7 SN74LVC245AN, U8 AE-LCNV4-MOSFET

Commit message: PCB V1.1
Parts:
- removed J4: PAL, IIeAux:PinHeader_1x02_P2.54mm_Horizontal, symbol IIeAux:Conn_01x02_Pin
- removed R1: 4K7, IIeAux:R_Axial_DIN0207_L6.3mm_D2.5mm_P10.16mm_Horizontal, symbol IIeAux:R
- removed R2: 0, IIeAux:R_Axial_DIN0207_L6.3mm_D2.5mm_P10.16mm_Horizontal, symbol IIeAux:R
- removed U8: AE-LCNV4-MOSFET, Apple2_bus:AE-LCNV4-MOSFET, symbol Apple2_bus:AE-LCNV4-MOSFET
- added C6: 0.1u, IIeAux:C_Disc_D4.3mm_W1.9mm_P5.08mm, symbol IIeAux:C
- added J2: Double Hi-Res, IIeAux:PinHeader_1x02_P2.54mm_Horizontal, symbol IIeAux:Conn_01x02_Pin
- added J3: PAL, IIeAux:PinHeader_1x02_P2.54mm_Horizontal, symbol IIeAux:Conn_01x02_Pin
- added R1: R, IIeAux:R_Axial_DIN0207_L6.3mm_D2.5mm_P10.16mm_Horizontal, symbol Apple2_bus:R
- added U2: SN74LVC245AN, IIeAux:DIP-20_W7.62mm_Socket, symbol IIeAux:SN74LVC245AN
- J1: value Apple IIe Aux -> Aux Slot
- U3: renamed from U5; footprint IIeAux:DIP-20_W7.62mm -> IIeAux:DIP-20_W7.62mm_Socket
- U4: renamed from U6; footprint IIeAux:DIP-20_W7.62mm -> IIeAux:DIP-20_W7.62mm_Socket
- U5: renamed from U1; footprint IIeAux:DIP-20_W7.62mm -> IIeAux:DIP-20_W7.62mm_Socket
- U8: renamed from U7; footprint IIeAux:DIP-20_W7.62mm -> IIeAux:DIP-20_W7.62mm_Socket
- renumbered C5 to C2, C2 to C4, C6 to C5, C4 to C7, C7 to C8, U2 to U1, U4 to U6, U3 to U7
Connections:
- net +3V3: now also C2.1, U5.1 (DIR), R1.1, U2.1 (DIR), U2.20 (VCC); no longer U4.1 (DIR)
- net +5V: now also C6.1; no longer C2.1
- net 14M: now also U8.8 (A7); no longer U8.9 (A8)
- net 80VID: now also U8.4 (A3); no longer U8.6 (A5)
- net AN3: now also U8.9 (A8), J2.2 (Pin_2); no longer U8.7 (A6)
- net C07X: now also U5.8 (A7)
- net D0: now also U4.2 (A1), U6.18 (D7); no longer U5.18 (B1), U6.3 (D0)
- net D1: now also U4.3 (A2), U6.17 (D6); no longer U5.17 (B2), U6.4 (D1)
- net D2: now also U4.4 (A3), U6.14 (D5); no longer U5.16 (B3), U6.7 (D2)
- net D3: now also U4.5 (A4), U6.13 (D4); no longer U5.15 (B4), U6.8 (D3)
- net D4: now also U4.6 (A5), U6.8 (D3); no longer U5.14 (B5), U6.13 (D4)
- net D5: now also U4.7 (A6), U6.7 (D2); no longer U5.13 (B6), U6.14 (D5)
- net D6: now also U4.8 (A7), U6.4 (D1); no longer U5.12 (B7), U6.17 (D6)
- net D7: now also U4.9 (A8), U6.3 (D0); no longer U5.11 (B8), U6.18 (D7)
- net EN80: now also U8.5 (A4); no longer U7.19 (CE)
- net FRCTXT: now also J2.1 (Pin_1)
- net GND: now also C6.2, J3.1 (Pin_1), U2.10 (GND); no longer U3.19 (~{OE})
- net GR: now also U5.2 (A1); no longer U8.5 (A4)
- net LDPS: now also U8.7 (A6)
- net PHI0: now also U8.2 (A1)
- net PHI1: now also U8.3 (A2)
- net PRAS: now also U5.7 (A6); no longer U8.2 (A1)
- net Q3: now also U5.5 (A4); no longer U8.3 (A2)
- net RA0: now also U2.2 (A1); no longer U3.2 (A1)
- net RA1: now also U2.3 (A2); no longer U3.3 (A2)
- net RA10: now also U5.3 (A2)
- net RA2: now also U2.4 (A3); no longer U3.4 (A3)
- net RA3: now also U2.5 (A4); no longer U3.5 (A4)
- net RA4: now also U2.6 (A5); no longer U3.6 (A5)
- net RA5: now also U2.7 (A6); no longer U3.7 (A6)
- net RA6: now also U2.8 (A7); no longer U3.8 (A7)
- net RA7: now also U2.9 (A8); no longer U3.9 (A8)
- net RA9: now also U5.4 (A3)
- net R/W: now also U5.9 (A8)
- net R/W80: now also U8.6 (A5); no longer U5.1 (DIR), U8.4 (A3)
- net SYNC: now also U5.6 (A5); no longer U8.8 (A7)
- net VID0: now also U3.9 (A8), U6.19 (O7); no longer U4.2 (A1), U6.2 (O0)
- net VID1: now also U3.8 (A7), U6.16 (O6); no longer U4.3 (A2), U6.5 (O1)
- net VID2: now also U3.7 (A6), U6.15 (O5); no longer U4.4 (A3), U6.6 (O2)
- net VID3: now also U3.6 (A5), U6.12 (O4); no longer U4.5 (A4), U6.9 (O3)
- net VID4: now also U3.5 (A4), U6.9 (O3); no longer U4.6 (A5), U6.12 (O4)
- net VID5: now also U3.4 (A3), U6.6 (O2); no longer U4.7 (A6), U6.15 (O5)
- net VID6: now also U3.3 (A2), U6.5 (O1); no longer U4.8 (A7), U6.16 (O6)
- net VID7: now also U3.2 (A1), U6.2 (O0); no longer U4.9 (A8), U6.19 (O7)
- net at U4.11 (B8): now also U1.27 (IOB15B_32); no longer U1.14 (35_IOB29A)
- net at U4.12 (B7): now also U1.28 (IOB15A_31); no longer U1.13 (40_IOB33B)
- net at U4.13 (B6): now also U1.29 (IOR24A_49); no longer U1.27 (IOB15B_32)
- net at U4.14 (B5): now also U1.30 (IOR24B_48); no longer U1.28 (IOB15A_31)
- net at U4.15 (B4): now also U1.38 (IOT37B_76); no longer U1.29 (IOR24A_49)
- net at U4.16 (B3): now also U1.39 (IOT37A_77); no longer U1.30 (IOR24B_48)
- net at U4.17 (B2): now also U1.13 (40_IOB33B); no longer U1.38 (IOT37B_76)
- net at U4.18 (B1): now also U1.14 (35_IOB29A); no longer U1.39 (IOT37A_77)
- net VID_EN: now reaches U1.2 (37_IOB31A)
- net VID_EN: now also U3.19 (~{OE})
- net RA_EN: now reaches U1.1 (38_IOB31B)
- net RA_EN: now also U2.19 (~{OE})
- net MD_EN: now reaches U1.4 (39_IOB33A)
- net MD_EN: now also U7.19 (CE)
- net D_R/W: now reaches U1.3 (36_IOB29B)
- net D_R/W: now also U4.1 (DIR)
- net at U1.5 (25_IOB8A): now also U5.18 (B1); no longer U5.2 (A1)
- net at U1.6 (26_IOB8B): now also U5.17 (B2); no longer U5.3 (A2)
- net at U1.7 (27_IOB11A): now also U5.16 (B3); no longer U5.4 (A3)
- net at U1.8 (28_IOB11B): now also U5.15 (B4); no longer U5.5 (A4)
- net at U1.9 (29_IOB13A): now also U5.14 (B5); no longer U5.6 (A5)
- net at U1.10 (30_IOB13B): now also U5.13 (B6); no longer U5.7 (A6)
- net at U1.11 (33_IOB23A): now also U5.12 (B7); no longer U5.8 (A7)
- net at U1.12 (34_IOB23B): now also U5.11 (B8); no longer U5.9 (A8)
- net at U1.48 (IOR5A_63): now also J3.2 (Pin_2), R1.2
- net A0: now reaches U1.40 (IOT12B_79), U3.11 (B8)
- net A0: now also U2.18 (B1)
- net A1: now reaches U1.41 (IOT12A_80), U3.12 (B7)
- net A1: now also U2.17 (B2)
- net A2: now reaches U1.42 (IOT11B_81), U3.13 (B6)
- net A2: now also U2.16 (B3)
- net A3: now reaches U1.43 (IOT11A_82), U3.14 (B5)
- net A3: now also U2.15 (B4)
- net A4: now reaches U1.44 (IOT10B_83), U3.15 (B4)
- net A4: now also U2.14 (B5)
- net A5: now reaches U1.45 (IOT10A_84), U3.16 (B3)
- net A5: now also U2.13 (B6)
- net A6: now reaches U1.46 (IOT8B_85), U3.17 (B2)
- net A6: now also U2.12 (B7)
- net A7: now reaches U1.47 (IOT8A_86), U3.18 (B1)
- net A7: now also U2.11 (B8)
- no-connect marks 27 -> 25
Other:
- moved on the sheet: C1, C2, C3, C4, C5, C7, C8, D1, J1, RN1, U1, U3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

Commit message: Use SEROUT signal
Connections:
- net LDPS: no longer U8.7 (A6)
- net SEROUT: now also U8.7 (A6)
Other:
- moved on the sheet: C6
Changed lines of the file:
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@@
 	(title_block
 		(title "IIeAux")
-		(date "2026-03-02")
-		(rev "1.1")
+		(date "2026-03-06")
+		(rev "1.2")
 		(company "nanja.info")
 		(comment 1 "Apple IIe Aux Slot FPGA Card")
+		(comment 2 "Use SEROUT signal")
 	)
 	(junction
@@
 	(wire
 		(pts
-			(xy 99.06 179.07) (xy 121.92 179.07)
+			(xy 110.49 179.07) (xy 121.92 179.07)
 		)
 		(stroke
@@
 	(wire
 		(pts
-			(xy 99.06 186.69) (xy 121.92 186.69)
+			(xy 110.49 186.69) (xy 121.92 186.69)
 		)
 		(stroke
@@
 		)
 	)
-	(global_label "LDPS"
+	(global_label "SEROUT"
 		(shape input)
 		(at 119.38 104.14 180)
@@
 		)
 		(property "Intersheetrefs" "${INTERSHEET_REFS}"
-			(at 111.6172 104.14 0)
+			(at 109.1377 104.14 0)
 			(effects
 				(font
@@
 	(symbol
 		(lib_id "IIeAux:C")
-		(at 99.06 182.88 0)
+		(at 110.49 182.88 0)
 		(unit 1)
 		(exclude_from_sim no)
@@
 		(fields_autoplaced yes)
 		(property "Reference" "C6"
-			(at 102.87 181.6099 0)
+			(at 114.3 181.6099 0)
 			(effects
 				(font
@@
 		)
 		(property "Value" "0.1u"
-			(at 102.87 184.1499 0)
+			(at 114.3 184.1499 0)
 			(effects
 				(font
@@
 		)
 		(property "Footprint" "IIeAux:C_Disc_D4.3mm_W1.9mm_P5.08mm"
-			(at 100.0252 186.69 0)
+			(at 111.4552 186.69 0)
 			(effects
 				(font
@@
 		)
 		(property "Datasheet" "~"
-			(at 99.06 182.88 0)
+			(at 110.49 182.88 0)
 			(effects
 				(font
@@
 		)
 		(property "Description" "Unpolarized capacitor"
-			(at 99.06 182.88 0)
+			(at 110.49 182.88 0)
 			(effects
 				(font

Commit message: V1.0 first batch
Parts:
- removed C6: 0.1u, IIeAux:C_Disc_D4.3mm_W1.9mm_P5.08mm, symbol IIeAux:C
- removed J3: PAL, IIeAux:PinHeader_1x02_P2.54mm_Horizontal, symbol IIeAux:Conn_01x02_Pin
- removed R1: R, IIeAux:R_Axial_DIN0207_L6.3mm_D2.5mm_P10.16mm_Horizontal, symbol Apple2_bus:R
- removed U2: SN74LVC245AN, IIeAux:DIP-20_W7.62mm_Socket, symbol IIeAux:SN74LVC245AN
- added J3: Aux, IIeAux:PinSocket_2x30_P2.54mm, symbol IIeAux:Conn_02x30_Counter_Clockwise
- added J4: PAL, IIeAux:PinHeader_1x02_P2.54mm_Horizontal, symbol IIeAux:Conn_01x02_Pin
- added J5: Y, IIeAux:PinSocket_1x08_P2.54mm_Vertical, symbol IIeAux:Conn_01x08
- added J6: X, IIeAux:PinSocket_1x08_P2.54mm_Vertical, symbol IIeAux:Conn_01x08
- added R1: 4K7, IIeAux:R_Axial_DIN0207_L6.3mm_D2.5mm_P10.16mm_Horizontal, symbol IIeAux:R
- J1: value Aux Slot -> Apple IIe Aux
- J2: value Double Hi-Res -> Double HiRes
- U1: renamed from U5; footprint IIeAux:DIP-20_W7.62mm_Socket -> IIeAux:DIP-20_W7.62mm
- U5: renamed from U3; footprint IIeAux:DIP-20_W7.62mm_Socket -> IIeAux:DIP-20_W7.62mm
- U6: renamed from U4; footprint IIeAux:DIP-20_W7.62mm_Socket -> IIeAux:DIP-20_W7.62mm
- U7: renamed from U8; footprint IIeAux:DIP-20_W7.62mm_Socket -> IIeAux:DIP-20_W7.62mm
- renumbered C4 to C2, C7 to C4, C2 to C5, C5 to C6, C8 to C7, D1 to D2, U1 to U2, U7 to U3, U6 to U4
Connections:
- net +3V3: now also U6.1 (DIR), R1.1; no longer C5.1, U1.1 (DIR)
- net +5V: now also C5.1, J3.30 (Pin_30)
- net 14M: now also J3.32 (Pin_32); no longer U7.8 (A7)
- net 3.58M: now also J3.1 (Pin_1)
- net 7M: now also J3.59 (Pin_59)
- net 80VID: now also J3.25 (Pin_25); no longer U7.4 (A3)
- net ALTVID: now also J3.27 (Pin_27)
- net AN3: now also J3.50 (Pin_50); no longer U7.9 (A8)
- net C07X: now also J3.6 (Pin_6); no longer U1.8 (A7)
- net CASEN: now also J3.37 (Pin_37)
- net CLRGAT: now also J3.24 (Pin_24)
- net D0: now also U1.2 (A1), U4.3 (D0); no longer U4.18 (D7), U6.2 (A1)
- net D1: now also U1.3 (A2), U4.4 (D1); no longer U4.17 (D6), U6.3 (A2)
- net D2: now also U1.4 (A3), U4.7 (D2); no longer U4.14 (D5), U6.4 (A3)
- net D3: now also U1.5 (A4), U4.8 (D3); no longer U4.13 (D4), U6.5 (A4)
- net D4: now also U1.6 (A5), U4.13 (D4); no longer U4.8 (D3), U6.6 (A5)
- net D5: now also U1.7 (A6), U4.14 (D5); no longer U4.7 (D2), U6.7 (A6)
- net D6: now also U1.8 (A7), U4.17 (D6); no longer U4.4 (D1), U6.8 (A7)
- net D7: now also U1.9 (A8), U4.18 (D7); no longer U4.3 (D0), U6.9 (A8)
- net EN80: now also U3.19 (CE), J3.26 (Pin_26); no longer U7.5 (A4)
- net ENTMG: now also J3.60 (Pin_60)
- net ENVID: now also J3.29 (Pin_29)
- net FRCTXT: now also J3.55 (Pin_55)
- net GND: now also U5.19 (~{OE}), J3.31 (Pin_31), J4.2 (Pin_2)
- net GR: now also J3.58 (Pin_58); no longer U1.2 (A1)
- net H0: now also J3.47 (Pin_47)
- net LDPS: now also J3.34 (Pin_34)
- net MD0: now also J3.44 (Pin_44)
- net MD1: now also J3.43 (Pin_43)
- net MD2: now also J3.40 (Pin_40)
- net MD3: now also J3.39 (Pin_39)
- net MD4: now also J3.21 (Pin_21)
- net MD5: now also J3.20 (Pin_20)
- net MD6: now also J3.17 (Pin_17)
- net MD7: now also J3.16 (Pin_16)
- net PCAS: now also J3.33 (Pin_33)
- net PHI0: now also J3.23 (Pin_23); no longer U7.2 (A1)
- net PHI1: now also J3.36 (Pin_36); no longer U7.3 (A2)
- net PRAS: now also J3.4 (Pin_4); no longer U1.7 (A6)
- net Q3: now also J3.53 (Pin_53); no longer U1.5 (A4)
- net RA0: now also U5.2 (A1), J3.51 (Pin_51)
- net RA1: now also U5.3 (A2), J3.10 (Pin_10)
- net RA10: now also J3.57 (Pin_57); no longer U1.3 (A2)
- net RA2: now also U5.4 (A3), J3.49 (Pin_49)
- net RA3: now also U5.5 (A4), J3.48 (Pin_48)
- net RA4: now also U5.6 (A5), J3.13 (Pin_13)
- net RA5: now also U5.7 (A6), J3.14 (Pin_14)
- net RA6: now also U5.8 (A7), J3.46 (Pin_46)
- net RA7: now also U5.9 (A8), J3.9 (Pin_9)
- net RA9: now also J3.56 (Pin_56); no longer U1.4 (A3)
- net ROMEN1: now also J3.11 (Pin_11)
- net ROMEN2: now also J3.12 (Pin_12)
- net R/W: now also U1.1 (DIR), J3.52 (Pin_52); no longer U1.9 (A8)
- net R/W80: now also J3.35 (Pin_35); no longer U7.6 (A5)
- net SEGA: now also J3.8 (Pin_8)
- net SEGB: now also J3.54 (Pin_54)
- net SEROUT: now also J3.28 (Pin_28); no longer U7.7 (A6)
- net SYNC: now also J3.3 (Pin_3); no longer U1.6 (A5)
- net VC: now also J3.5 (Pin_5)
- net VID0: now also U4.2 (O0), J3.45 (Pin_45); no longer U4.19 (O7), U5.9 (A8)
- net VID1: now also U4.5 (O1), J3.42 (Pin_42); no longer U4.16 (O6), U5.8 (A7)
- net VID2: now also U4.6 (O2), J3.41 (Pin_41); no longer U4.15 (O5), U5.7 (A6)
- net VID3: now also U4.9 (O3), J3.38 (Pin_38); no longer U4.12 (O4), U5.6 (A5)
- net VID4: now also U4.12 (O4), J3.22 (Pin_22); no longer U4.9 (O3), U5.5 (A4)
- net VID5: now also U4.15 (O5), J3.19 (Pin_19); no longer U4.6 (O2), U5.4 (A3)
- net VID6: now also U4.16 (O6), J3.18 (Pin_18); no longer U4.5 (O1), U5.3 (A2)
- net VID7: now also U4.19 (O7), J3.15 (Pin_15); no longer U4.2 (O0), U5.2 (A1)
- net VID7M: now also J3.2 (Pin_2)
- net WNDW: now also J3.7 (Pin_7)
- net at U2.48 (IOR5A_63): now also J4.1 (Pin_1), R1.2
- net at U6.11 (B8): now also U2.14 (35_IOB29A); no longer U2.27 (IOB15B_32)
- net at U6.12 (B7): now also U2.13 (40_IOB33B); no longer U2.28 (IOB15A_31)
- net at U6.13 (B6): now also U2.27 (IOB15B_32); no longer U2.29 (IOR24A_49)
- net at U6.14 (B5): now also U2.28 (IOB15A_31); no longer U2.30 (IOR24B_48)
- net at U6.15 (B4): now also U2.29 (IOR24A_49); no longer U2.38 (IOT37B_76)
- net at U6.16 (B3): now also U2.30 (IOR24B_48); no longer U2.39 (IOT37A_77)
- net at U6.17 (B2): now also U2.38 (IOT37B_76); no longer U2.13 (40_IOB33B)
- net at U6.18 (B1): now also U2.39 (IOT37A_77); no longer U2.14 (35_IOB29A)
- net A0: no longer names the net of U2.40 (IOT12B_79), U5.11 (B8)
- net A1: no longer names the net of U2.41 (IOT12A_80), U5.12 (B7)
- net A2: no longer names the net of U2.42 (IOT11B_81), U5.13 (B6)
- net A3: no longer names the net of U2.43 (IOT11A_82), U5.14 (B5)
- net A4: no longer names the net of U2.44 (IOT10B_83), U5.15 (B4)
- net A5: no longer names the net of U2.45 (IOT10A_84), U5.16 (B3)
- net A6: no longer names the net of U2.46 (IOT8B_85), U5.17 (B2)
- net A7: no longer names the net of U2.47 (IOT8A_86), U5.18 (B1)
- net D_R/W: no longer names the net of U2.3 (36_IOB29B)
- net D_R/W: no longer U6.1 (DIR)
- net MD_EN: no longer names the net of U2.4 (39_IOB33A)
- net MD_EN: no longer U3.19 (CE)
- net RA_EN: no longer names the net of U2.1 (38_IOB31B)
- net VID_EN: no longer names the net of U2.2 (37_IOB31A)
- net VID_EN: no longer U5.19 (~{OE})
- new net X0: J6.1 (Pin_1), U6.2 (A1)
- new net X1: J6.2 (Pin_2), U6.3 (A2)
- new net X2: J6.3 (Pin_3), U6.4 (A3)
- new net X3: J6.4 (Pin_4), U6.5 (A4)
- new net X4: J6.5 (Pin_5), U6.6 (A5)
- new net X5: J6.6 (Pin_6), U6.7 (A6)
- new net X6: J6.7 (Pin_7), U6.8 (A7)
- new net X7: J6.8 (Pin_8), U6.9 (A8)
- new net Y0: J5.1 (Pin_1), U7.2 (A1)
- new net Y1: J5.2 (Pin_2), U7.3 (A2)
- new net Y2: J5.3 (Pin_3), U7.4 (A3)
- new net Y3: J5.4 (Pin_4), U7.5 (A4)
- new net Y4: J5.5 (Pin_5), U7.6 (A5)
- new net Y5: J5.6 (Pin_6), U7.7 (A6)
- new net Y6: J5.7 (Pin_7), U7.8 (A7)
- new net Y7: J5.8 (Pin_8), U7.9 (A8)
- no-connect marks 25 -> 12
Other:
- moved on the sheet: C1, C2, C3, C4, C5, C6, C7, D2, RN1, U1, U2, U3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

Commit message: fixed U1 direction
Connections:
- net D0: now also U1.18 (B1); no longer U1.2 (A1)
- net D1: now also U1.17 (B2); no longer U1.3 (A2)
- net D2: now also U1.16 (B3); no longer U1.4 (A3)
- net D3: now also U1.15 (B4); no longer U1.5 (A4)
- net D4: now also U1.14 (B5); no longer U1.6 (A5)
- net D5: now also U1.13 (B6); no longer U1.7 (A6)
- net D6: now also U1.12 (B7); no longer U1.8 (A7)
- net D7: now also U1.11 (B8); no longer U1.9 (A8)
- net R/W: no longer U1.1 (DIR)
- net R/W80: now also U1.1 (DIR)
- net at U2.12 (34_IOB23B): now also U1.9 (A8); no longer U1.11 (B8)
- net at U2.11 (33_IOB23A): now also U1.8 (A7); no longer U1.12 (B7)
- net at U2.10 (30_IOB13B): now also U1.7 (A6); no longer U1.13 (B6)
- net at U2.9 (29_IOB13A): now also U1.6 (A5); no longer U1.14 (B5)
- net at U2.8 (28_IOB11B): now also U1.5 (A4); no longer U1.15 (B4)
- net at U2.7 (27_IOB11A): now also U1.4 (A3); no longer U1.16 (B3)
- net at U2.6 (26_IOB8B): now also U1.3 (A2); no longer U1.17 (B2)
- net at U2.5 (25_IOB8A): now also U1.2 (A1); no longer U1.18 (B1)
Changed lines of the file:
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@@
 	(title_block
 		(title "IIeAux")
-		(date "2025-05-05")
+		(date "2026-03-07")
 		(rev "1")
 		(company "nanja.info")
+		(comment 1 "fixed U1 direction")
 	)
 	(junction
@@
 	(wire
 		(pts
-			(xy 157.48 43.18) (xy 162.56 43.18)
+			(xy 132.08 43.18) (xy 124.46 43.18)
 		)
 		(stroke
@@
 	(wire
 		(pts
-			(xy 162.56 43.18) (xy 162.56 44.45)
+			(xy 124.46 43.18) (xy 124.46 44.45)
 		)
 		(stroke
@@
 	(wire
 		(pts
-			(xy 130.81 43.18) (xy 132.08 43.18)
-		)
-		(stroke
-			(width 0)
-			(type default)
-		)
-	)
-	(wire
-		(pts
 			(xy 92.71 55.88) (xy 91.44 55.88)
 		)
@@
 	(wire
 		(pts
+			(xy 160.02 43.18) (xy 157.48 43.18)
+		)
+		(stroke
+			(width 0)
+			(type default)
+		)
+	)
+	(wire
+		(pts
 			(xy 269.24 137.16) (xy 267.97 137.16)
 		)
@@
 		)
 	)
-	(global_label "R{slash}W"
+	(global_label "R{slash}W80"
 		(shape input)
-		(at 130.81 43.18 180)
+		(at 160.02 43.18 0)
 		(fields_autoplaced yes)
 		(effects
@@
 				(size 1.27 1.27)
 			)
-			(justify right)
+			(justify left)
 		)
 		(property "Intersheetrefs" "${INTERSHEET_REFS}"
-			(at 123.7729 43.18 0)
+			(at 169.4761 43.18 0)
 			(effects
 				(font
 					(size 1.27 1.27)
 				)
-				(justify right)
+				(justify left)
 				(hide yes)
 			)
@@
 	(symbol
 		(lib_id "IIeAux:GND")
-		(at 162.56 44.45 0)
+		(at 124.46 44.45 0)
+		(mirror y)
 		(unit 1)
 		(exclude_from_sim no)
@@
 		(dnp no)
 		(property "Reference" "#PWR014"
-			(at 162.56 50.8 0)
+			(at 124.46 50.8 0)
 			(effects
 				(font
@@
 		)
 		(property "Value" "GND"
-			(at 166.37 46.99 0)
+			(at 120.65 46.99 0)
 			(effects
 				(font
@@
 		)
 		(property "Footprint" ""
-			(at 162.56 44.45 0)
+			(at 124.46 44.45 0)
 			(effects
 				(font
@@
 		)
 		(property "Datasheet" ""
-			(at 162.56 44.45 0)
+			(at 124.46 44.45 0)
 			(effects
 				(font
@@
 		)
 		(property "Description" "Power symbol creates a global label with name \"GND\" , ground"
-			(at 162.56 44.45 0)
+			(at 124.46 44.45 0)
 			(effects
 				(font
@@
 		(lib_id "IIeAux:SN74LVC245AN")
 		(at 144.78 53.34 0)
+		(mirror y)
 		(unit 1)
 		(exclude_from_sim no)
@@
 		(on_board yes)
 		(dnp no)
-		(fields_autoplaced yes)
 		(property "Reference" "U1"
-			(at 146.9233 33.02 0)
+			(at 142.6367 33.02 0)
 			(effects
 				(font
@@
 		)
 		(property "Value" "SN74LVC245AN"
-			(at 146.9233 35.56 0)
+			(at 142.6367 35.56 0)
 			(effects
 				(font
@@
 		)
 		(property "Footprint" "IIeAux:DIP-20_W7.62mm"
-			(at 167.64 69.85 0)
+			(at 121.92 69.85 0)
 			(effects
 				(font
@@
 		)
 		(property "Datasheet" "https://www.ti.com/lit/ds/scas218x/scas218x.pdf"
-			(at 143.51 59.69 0)
+			(at 146.05 59.69 0)
 			(effects
 				(font
